Commit message: Add Gazebo differential drive robot

File: src/urdf_demo/urdf/robot.urdf (robot description, URDF)
Before this commit: robot my_robot, 2 links, 1 joints
Links:
- added link left_wheel, mass 0.5; collision cylinder length=0.08 radius=0.15; visual cylinder length=0.08 radius=0.15
- added link right_wheel, mass 0.5; collision cylinder length=0.08 radius=0.15; visual cylinder length=0.08 radius=0.15
- link base_link: mass None -> 5.0; geometry collision box size=1.0 0.6 0.3; visual box size=1.0 0.6 0.3
- link sensor_link: mass None -> 0.5; geometry collision cylinder length=0.2 radius=0.1; visual cylinder length=0.2 radius=0.1
Joints:
- added joint left_wheel_joint: type continuous, parent base_link, child left_wheel, origin xyz=0 0.35 -0.05 rpy=1.5708 0 0, axis 0 0 1
- added joint right_wheel_joint: type continuous, parent base_link, child right_wheel, origin xyz=0 -0.35 -0.05 rpy=1.5708 0 0, axis 0 0 1

Commit message: Add Gazebo LiDAR sensor integration

File: src/urdf_demo/urdf/robot.urdf (robot description, URDF)
Before this commit: robot my_robot, 4 links, 3 joints
Links:
- link sensor_link: geometry visual cylinder length=0.2 radius=0.1
